File: schematics/rc-miata.kicad_pcb (KiCad board)
At the start: 2 copper layers, 2 parts, among them U1 ESP32-C3-DevKitM-1, U2 LM7805_TO220

Commit message: Updated header blocks. Populated PCB title block
Parts:
- removed U1: ESP32-C3-DevKitM-1, RF_Module:ESP32-C3-DevKitM-1
- removed U2: LM7805_TO220, Package_TO_SOT_THT:TO-220-3_Vertical
Routing:
- net +5V: track 40.1 -> 0.00 mm
- net GND: track 38.3 -> 0.00 mm
