File: schematics/rc-miata.kicad_pcb (KiCad board)
At the start: 2 copper layers, 0 parts

Commit message: Rough PCB layout. Basic board properties
Parts:
- added C1: 100n, Capacitor_SMD:C_0603_1608Metric_Pad1.08x0.95mm_HandSolder, F.Cu at (163.9, 113.5)
- added D1: YELLOW, LED_THT:LED_D3.0mm, F.Cu at (109.0, 173.6)
- added D2: YELLOW, LED_THT:LED_D3.0mm, F.Cu at (109.0, 179.1)
- added D3: RED, LED_THT:LED_D3.0mm, F.Cu at (109.0, 184.5)
- added D4: YELLOW, LED_THT:LED_D3.0mm, F.Cu at (109.0, 190.0)
- added H1: M3, MountingHole:MountingHole_3.2mm_M3_Pad_Via, F.Cu at (214.3, 50.8)
- added H2: M3, MountingHole:MountingHole_3.2mm_M3_Pad_Via, F.Cu at (108.8, 55.2)
- added H3: M3, MountingHole:MountingHole_3.2mm_M3_Pad_Via, F.Cu at (109.6, 148.5)
- added H4: M3, MountingHole:MountingHole_3.2mm_M3_Pad_Via, F.Cu at (204.0, 154.6)
- added J1: Battery, Connectors:1869211, F.Cu at (144.9, 127.5)
- added J2: Switch, Connectors:1869211, F.Cu at (161.9, 128.5)
- added J3: UBEC, Connectors:1161181, F.Cu at (196.0, 135.2)
- added J4: ESC, Connectors:1869237, F.Cu at (196.0, 105.3)
- added J5: SERVO, Connectors:1161181, F.Cu at (195.5, 74.7)
- added R1: 330, Resistor_THT:R_Axial_DIN0204_L3.6mm_D1.6mm_P5.08mm_Horizontal, F.Cu at (137.4, 175.5)
- added R2: 330, Resistor_THT:R_Axial_DIN0204_L3.6mm_D1.6mm_P5.08mm_Horizontal, F.Cu at (137.4, 178.7)
- added U3: ESP32, ESP32:ESP32 Devkitv1, F.Cu at (123.5, 112.2)
